Commit message: Adjusted the initial gesture to open.

File: urdf/rohand_left.urdf (robot description, URDF)
Before this commit: robot rohand_left, 26 links, 25 joints
Links:
- link base_link: mass 0.0407795398922086 -> 0.0556275033895707
- link if_connecting_link: mass 0.000200341201168555 -> 0.000200341201168535
- link if_distal_link: mass 0.000118307873360847 -> 0.00606060335159451
- link if_proximal_link: mass 0.00193521128531993 -> 0.00193519028805872
- link if_slider_abpart_link: mass 0.000420491610160664 -> 0.000420484116155222
- link if_slider_link: mass 0.000489108023003754 -> 0.000489121771249986
- link lf_connecting_link: mass 0.000176992753343057 -> 0.000176992753343061
- link lf_distal_link: mass 0.000118307873360846 -> 0.00364905952774006
- link lf_proximal_link: mass 0.00177912026577765 -> 0.00177911361510511
- link lf_slider_abpart_link: mass 0.000420491508642964 -> 0.000420507370337398
- link lf_slider_link: mass 0.000489106181447385 -> 0.00048912103124811
- link mf_connecting_link: mass 0.000215108926153008 -> 0.000215108931947231
- link mf_distal_link: mass 0.000118307873360846 -> 0.00606061622476954
- link mf_proximal_link: mass 0.00237723145934376 -> 0.00237722144967564
- link mf_slider_abpart_link: mass 0.000420491400161604 -> 0.000420507611933596
- link mf_slider_link: mass 0.000489123101663119 -> 0.000489119216361822
- link rf_connecting_link: mass 0.000200341201168549 -> 0.000200341201168546
- link rf_distal_link: mass 0.000118307873360846 -> 0.00606025074073705
- link rf_proximal_link: mass 0.00193531294665337 -> 0.00193520497103009
- link rf_slider_abpart_link: mass 0.000420491416628446 -> 0.000420484347510521
- link rf_slider_link: mass 0.00048912323990742 -> 0.000489121716234798
- link th_connecting_link: mass 0.000337391699812154 -> 0.000337394683077766
- link th_distal_link: mass 0.00014720241261084 -> 0.00398421921008986
- link th_proximal_link: mass 0.0054430978910106 -> 0.00544482144605495
- link th_root_link: mass 0.00208321489353089 -> 0.00219012478679673
- link th_slider_link: mass 0.00164989215630923 -> 0.00096692626401777
Joints:
- joint if_connecting_link: axis 1 0 0 -> 0 1 0; origin xyz=0.034369 0.1159 0.032401 rpy=-0.0048911 0.098868 -0.049512 -> xyz=-0.11999 0.035982 0.0028163 rpy=-0.087248 -0.0072243 -0.082404
- joint if_distal_link: axis 1 0 0 -> 0 1 0; origin xyz=0 0.035719 -0.0037924 rpy=0 0 0 -> xyz=-0.035842 0 -0.0023622 rpy=0 0 0
- joint if_proximal_link: axis 1 0 0 -> 0 1 0; origin xyz=0.036159 0.10951 0.026256 rpy=-0.0048911 0.098868 -0.049512 -> xyz=-0.1124 0.037665 -0.0018024 rpy=-0.087248 -0.0072243 -0.082404
- joint if_slider_abpart_link: axis -1 0 0 -> 0 1 0; origin xyz=0.003488 -0.029 0.00029936 rpy=0.22394 0.085779 -3.1416 -> xyz=-0.029 0.0034859 -0.00030434 rpy=-0.087248 -0.0072243 0.0006319
- joint if_slider_link: axis 0 1 0 -> 1 0 0; limit lower=-0.003 upper=0.016 effort=0 velocity=0 -> lower=0 upper=0.019 effort=0 velocity=0; origin xyz=0.025508 0.071777 0.0097223 rpy=-2.9236 0.01514 -0.068245 -> xyz=-0.074388 0.026652 -0.009751 rpy=0 0 -0.083036
- joint lf_connecting_link: axis 1 0 0 -> 0 1 0; origin xyz=-0.027992 0.11241 0.033343 rpy=-0.012586 -0.11505 0.10921 -> xyz=-0.11722 -0.02643 0.0045821 rpy=0.087265 -0.010332 0.11755
- joint lf_distal_link: axis 1 0 0 -> 0 1 0; origin xyz=0 0.031591 -0.0046466 rpy=0 0 0 -> xyz=-0.03178 0 -0.0031085 rpy=0 0 0
- joint lf_proximal_link: axis 1 0 0 -> 0 1 0; origin xyz=-0.023967 0.10652 0.027793 rpy=-0.012586 -0.11505 0.10921 -> xyz=-0.11021 -0.022502 0.0004348 rpy=0.087265 -0.010332 0.11755
- joint lf_slider_abpart_link: axis -1 0 0 -> 0 1 0; origin xyz=0.003487 -0.029 -0.00031085 rpy=0.23027 -0.088748 -3.1416 -> xyz=-0.029 0.0034858 0.00030556 rpy=0.087277 -0.010237 -0.0008957
- joint lf_slider_link: axis 0 1 0 -> 1 0 0; limit lower=-0.003 upper=0.016 effort=0 velocity=0 -> lower=0 upper=0.019 effort=0 velocity=0; origin xyz=-0.024745 0.06733 0.0096888 rpy=-2.9253 -0.02839 0.12847 -> xyz=-0.070738 -0.024172 -0.0087474 rpy=-1.1295E-05 -9.4916E-05 0.11844
- joint mf_connecting_link: axis 1 0 0 -> 0 1 0; origin xyz=0.01345 0.11796 0.037645 rpy=0 -0.001438 -0.00032101 -> xyz=-0.12312 0.015086 0.0075148 rpy=-5.1083E-05 0 -0.013233
- joint mf_distal_link: axis 1 0 0 -> 0 1 0; origin xyz=0 0.040599 -0.0057752 rpy=0 0 0 -> xyz=-0.040918 0 -0.0027058 rpy=0 0 0
- joint mf_proximal_link: axis 1 0 0 -> 0 1 0; origin xyz=0.016157 0.11167 0.031745 rpy=0 -0.001438 -0.00032101 -> xyz=-0.11567 0.017687 0.0031149 rpy=-5.1083E-05 0 -0.013233
- joint mf_slider_abpart_link: axis -1 0 0 -> 0 1 0; origin xyz=0.0035008 -0.029 0 rpy=0.2183 -0.0013907 -3.1416 -> xyz=-0.029 0.0034992 0 rpy=-5.1711E-05 4.6769E-05 0
- joint mf_slider_link: axis 0 1 0 -> 1 0 0; limit lower=-0.003 upper=0.016 effort=0 velocity=0 -> lower=0 upper=0.019 effort=0 velocity=0; origin xyz=0.0090697 0.072773 0.014291 rpy=-2.9233 0 1.4106E-05 -> xyz=-0.076966 0.010074 -0.0054828 rpy=0 -4.7445E-05 -0.013233
- joint rf_connecting_link: axis 1 0 0 -> 0 1 0; origin xyz=-0.0070772 0.11568 0.036339 rpy=-0.0011254 -0.016556 0.067871 -> xyz=-0.12089 -0.0054721 0.0067674 rpy=-7.9422E-05 0 0.056583
- joint rf_distal_link: axis 1 0 0 -> 0 1 0; origin xyz=0 0.035597 -0.0048092 rpy=0 0 0 -> xyz=-0.035824 0 -0.0026256 rpy=0 0 0
- joint rf_proximal_link: axis 1 0 0 -> 0 1 0; origin xyz=-0.0038595 0.10959 0.030486 rpy=-0.0011254 -0.016556 0.067871 -> xyz=-0.11363 -0.0023572 0.0023678 rpy=-7.9422E-05 0 0.056583
- joint rf_slider_abpart_link: axis -1 0 0 -> 0 1 0; origin xyz=0.0035008 -0.029 0 rpy=0.21881 -0.0013941 -3.1416 -> xyz=-0.029 0.0034992 0 rpy=-7.4035E-05 9.9598E-05 0
- joint rf_slider_link: axis 0 1 0 -> 1 0 0; limit lower=-0.003 upper=0.016 effort=0 velocity=0 -> lower=0 upper=0.019 effort=0 velocity=0; origin xyz=-0.0080245 0.070447 0.012986 rpy=-2.9239 -0.015105 0.068179 -> xyz=-0.074491 -0.0072514 -0.0062279 rpy=0 -9.51E-05 0.056583
- joint th_connecting_link: axis 0 0 -1 -> 0 0 1; origin xyz=-0.00079692 -0.0341 0.0042568 rpy=-0.12733 0.56582 2.9072 -> xyz=0.0333 0.0003242 0.00399 rpy=-0.032033 -0.02575 -0.67687
- joint th_distal_link: origin xyz=-0.00015706 0.057513 -0.00075 rpy=0 0 0 -> xyz=-0.046968 0.023498 0.002 rpy=3.1416 0 3.1416
- joint th_proximal_link: axis 0 0 1 -> 0 0 -1; origin xyz=0.012034 -0.028305 0.020114 rpy=-0.00017213 0.56949 3.1413 -> xyz=-0.028155 0.021344 -0.011022 rpy=0.032033 -0.00041454 0.012934
- joint th_root_link: axis 0 -1 0 -> -1 0 0; limit lower=-0.785 upper=0.785 effort=0 velocity=0 -> lower=0 upper=1.57 effort=0 velocity=0; origin xyz=0.019264 0.028865 -0.012597 rpy=3.1416 0 -0.00031701 -> xyz=-0.025192 0.019558 -0.022233 rpy=0.0028708 -0.21841 -0.013249
- joint th_slider_link: axis 0 -1 0 -> 1 0 0; limit lower=-0.003 upper=0.003 effort=0 velocity=0 -> lower=0 upper=0.01 effort=0 velocity=0; origin xyz=-0.0033135 0.014022 -0.0077 rpy=0 0.57844 -2.9442 -> xyz=-0.0038117 0.0056317 0.00895 rpy=-3.1005 0 2.4643

File: urdf/rohand_right.urdf (robot description, URDF)
Before this commit: robot rohand_right, 26 links, 25 joints
Links:
- link base_link: mass 0.0490769144926836 -> 0.0567346930426757
- link if_connecting_link: mass 0.00020034120116847 -> 0.000200341201166992
- link if_distal_link: mass 0.000118307873360846 -> 0.00606035931095405
- link if_proximal_link: mass 0.00193522991741753 -> 0.00193554425496127
- link if_slider_abpart_link: mass 0.000420506796259996 -> 0.000420484339978023
- link if_slider_link: mass 0.000489112297930526 -> 0.00048910557498402
- link lf_connecting_link: mass 0.000176992753343061 -> 0.000176992753343264
- link lf_distal_link: mass 0.000118307873360846 -> 0.00177085221629863
- link lf_proximal_link: mass 0.00177930732045757 -> 0.00177920059071157
- link lf_slider_abpart_link: mass 0.000420506872592595 -> 0.000420484114077754
- link lf_slider_link: mass 0.000489116937789504 -> 0.000489105121519416
- link mf_connecting_link: mass 0.000215109025045747 -> 0.000215117295970291
- link mf_distal_link: mass 0.000118307873360846 -> 0.00606075827170448
- link mf_proximal_link: mass 0.0023771786956887 -> 0.00237749526593246
- link mf_slider_abpart_link: mass 0.000420506980543982 -> 0.000420484349049402
- link mf_slider_link: mass 0.000489115418477034 -> 0.000489105694012057
- link rf_connecting_link: mass 0.000200341201168546 -> 0.000200341201166998
- link rf_distal_link: mass 0.000118307873360846 -> 0.00606084017975732
- link rf_proximal_link: mass 0.00193520051388196 -> 0.00193555006791898
- link rf_slider_abpart_link: mass 0.000420506921107561 -> 0.000420484118672501
- link rf_slider_link: mass 0.000489115404099442 -> 0.000489105700009114
- link th_connecting_link: mass 0.000337391875240177 -> 0.00033738169009293
- link th_distal_link: mass 0.000147202412610839 -> 0.00247307051858648
- link th_proximal_link: mass 0.00544330421208834 -> 0.00544486421565137
- link th_root_link: mass 0.0733985032398848 -> 0.00217787514894826
- link th_slider_link: mass 0.00164989230216945 -> 0.000966922791670203
Joints:
- joint if_connecting_link: origin xyz=-0.11996 -0.036476 0.0065579 rpy=0.087248 -0.0072339 0.082513 -> xyz=-0.12072 -0.027274 0.0035849 rpy=0.087248 -0.0072339 0.082513
- joint if_distal_link: origin xyz=-0.034068 0 -0.011383 rpy=0 0 0 -> xyz=-0.035842 -0.00039995 -0.0023622 rpy=0 0 0
- joint if_proximal_link: origin xyz=-0.11237 -0.038159 0.0019394 rpy=0.087248 -0.0072339 0.082513 -> xyz=-0.11362 -0.023198 -0.00052831 rpy=0.087248 -0.0072339 0.082513
- joint if_slider_abpart_link: origin xyz=-0.029 -0.0034875 -0.00030444 rpy=0.087237 -0.007223 -0.00063172 -> xyz=-0.029 0.0034858 0.00030547 rpy=0.087249 -0.0072239 -0.00063188
- joint if_slider_link: limit lower=-0.003 upper=0.016 effort=0 velocity=0 -> lower=0 upper=0.019 effort=0 velocity=0; origin xyz=-0.071835 -0.02643 -0.0059651 rpy=0 0 0.083145 -> xyz=-0.074395 -0.026674 -0.0097486 rpy=0 0 0.083145
- joint lf_connecting_link: origin xyz=-0.11738 0.02595 0.0084121 rpy=-0.087265 -0.01032 -0.11741 -> xyz=-0.11629 0.03512 0.0038182 rpy=-0.087265 -0.01032 -0.11741
- joint lf_distal_link: origin xyz=-0.029816 0 -0.011429 rpy=0 0 0 -> xyz=-0.03178 0 -0.0031085 rpy=0 0 0
- joint lf_proximal_link: origin xyz=-0.11038 0.022023 0.0042647 rpy=-0.087265 -0.01032 -0.11741 -> xyz=-0.10865 0.036534 -0.00079985 rpy=-0.087265 -0.01032 -0.11741
- joint lf_slider_abpart_link: origin xyz=-0.029 -0.0034874 0.00030573 rpy=-0.087286 -0.010238 0.00089593 -> xyz=-0.029 0.0034859 -0.00030443 rpy=-0.087275 -0.010237 0.00089571
- joint lf_slider_link: limit lower=-0.003 upper=0.016 effort=0 velocity=0 -> lower=0 upper=0.019 effort=0 velocity=0; origin xyz=-0.068152 0.023874 -0.0049615 rpy=0 -8.2704E-05 -0.11831 -> xyz=-0.070846 0.024164 -0.0087451 rpy=0 -8.2704E-05 -0.11831
- joint mf_connecting_link: origin xyz=-0.12313 -0.015578 0.011298 rpy=7.2594E-05 0 0.013228 -> xyz=-0.12325 -0.0063087 0.007515 rpy=7.2594E-05 0 0.013228
- joint mf_distal_link: origin xyz=-0.038382 0 -0.014438 rpy=0 0 0 -> xyz=-0.040918 0 -0.0027079 rpy=0 0 0
- joint mf_proximal_link: origin xyz=-0.11567 -0.018179 0.0068982 rpy=7.2594E-05 0 0.013228 -> xyz=-0.11587 -0.0035104 0.0031158 rpy=7.2594E-05 0 0.013228
- joint mf_slider_abpart_link: origin xyz=-0.029 -0.0035008 0 rpy=6.1564E-05 9.9576E-05 0 -> xyz=-0.029 0.0034992 0 rpy=7.3922E-05 9.943E-05 0
- joint mf_slider_link: limit lower=-0.003 upper=0.016 effort=0 velocity=0 -> lower=0 upper=0.019 effort=0 velocity=0; origin xyz=-0.074014 -0.010026 -0.001697 rpy=0 -0.00010039 0.013228 -> xyz=-0.076975 -0.010095 -0.0054807 rpy=0 -0.00010039 0.013228
- joint rf_connecting_link: origin xyz=-0.12092 0.0049808 0.010553 rpy=7.942E-05 0 -0.056587 -> xyz=-0.1204 0.014236 0.0067704 rpy=7.942E-05 0 -0.056587
- joint rf_distal_link: origin xyz=-0.033703 0 -0.012425 rpy=0 0 0 -> xyz=-0.035824 0 -0.0026256 rpy=0 0 0
- joint rf_proximal_link: origin xyz=-0.11367 0.0018657 0.0061535 rpy=7.942E-05 0 -0.056587 -> xyz=-0.11283 0.016512 0.0023712 rpy=7.942E-05 0 -0.056587
- joint rf_slider_abpart_link: origin xyz=-0.029 -0.0035008 0 rpy=6.3004E-05 9.8956E-05 0 -> xyz=-0.029 0.0034992 0 rpy=7.4034E-05 9.9581E-05 0
- joint rf_slider_link: limit lower=-0.003 upper=0.016 effort=0 velocity=0 -> lower=0 upper=0.019 effort=0 velocity=0; origin xyz=-0.071688 0.0071015 -0.0024419 rpy=0 -9.5082E-05 -0.056587 -> xyz=-0.074498 0.0072308 -0.0062256 rpy=0 -9.5082E-05 -0.056587
- joint th_connecting_link: axis 0 0 -1 -> 0 1 0; origin xyz=-0.0340999999274571 -0.00309060345004721 -0.0037899565057163 rpy=-0.335166812648025 -0.0427408662491538 -0.122062712839907 -> xyz=0.0333 0 -0.0040032 rpy=-1.603 0.025523 -2.4719
- joint th_distal_link: axis 0 0 1 -> 0 1 0; origin xyz=0.057388 0.0037551 5E-05 rpy=3.1416 0 3.1416 -> xyz=0.046968 -0.023498 -0.0139 rpy=-1.5708 0 3.1345
- joint th_proximal_link: origin xyz=-0.028307 -0.023252 -0.0029666 rpy=-2.8064 0.0045041 3.1287 -> xyz=-0.028155 -0.021306 -0.0089619 rpy=-3.1067 0.00045151 3.1287
- joint th_root_link: origin xyz=-0.025193 -0.019549 -0.018448 rpy=-0.00287 -0.21841 0.013245 -> xyz=-0.025193 -0.01958 -0.022231 rpy=0 -0.21841 0.013245
- joint th_slider_link: axis -1 0 0 -> 1 0 0; limit lower=-0.003 upper=0.003 effort=0 velocity=0 -> lower=0 upper=0.01 effort=0 velocity=0; origin xyz=0.014212 -0.0023514 -0.0077 rpy=-2.8038 0 3.0123 -> xyz=0.0038117 -0.0056317 -0.00695 rpy=-0.041099 0 -0.67728
