Commit message: fix th_slider_link form 0-0.0007 to 0-0.010

File: ap002/urdf/rohand_left.urdf (robot description, URDF)
Before this commit: robot rohand_left, 26 links, 25 joints
Joints:
- joint th_slider_link: limit lower=0 upper=0.007 effort=0 velocity=0 -> lower=0 upper=0.010 effort=0 velocity=0

File: ap002/urdf/rohand_right.urdf (robot description, URDF)
Before this commit: robot rohand_right, 26 links, 25 joints
Joints:
- joint th_slider_link: limit lower=0 upper=0.007 effort=0 velocity=0 -> lower=0 upper=0.010 effort=0 velocity=0
